File: hardware/PCB/glassify/glassify.kicad_pcb (KiCad board)
At the start: 2 copper layers, 61 x 58 mm, 16 parts, among them J1 Conn_02x09_Odd_Even

Commit message: Final update to hardware - PCBs & Datasheets
Parts:
- removed POWER: 2mm_pitch, Connector_Molex:Molex_KK-254_AE-6410-02A_1x02_P2.54mm_Vertical
- added J2: Conn_01x03_Male, GLFfootprints:power_adapter_conn, F.Cu at (175.5, 97.5)
- moved LEDs 6.56 mm to (167.5, 92.5)
- moved BD137G 0.10 mm to (157.5, 89.0)
- renumbered 1206A_1 to 1206A, 1206A_02 to 1206A
Connections:
- J1 pad 11: Net-(1206A_01x08_Male1-Pad5) -> Net-(2mm_pitch4-Pad1)
- J1 pad 2: Net-(J1-Pad1) -> Net-(J1-Pad2)
- J1 pad 6: Net-(2mm_pitch4-Pad1) -> Net-(BD137G1-Pad3)
- J1 pad 8: Net-(BD137G1-Pad3) -> Net-(1206A_01x08_Male1-Pad5)
Routing:
- net Net-(BD137G1-Pad2): track 8.56 -> 30.5 mm
- net Net-(1206A_01x08_Male1-Pad5): track 49.8 -> 37.9 mm
- net Net-(BD137G1-Pad3): track 44.5 -> 36.7 mm
- net Net-(2mm_pitch4-Pad1): track 35.4 -> 29.6 mm
- net Net-(2mm_pitch4-Pad2): track 24.6 -> 21.5 mm, vias 0 -> 1
- net Net-(2mm_pitch4-Pad3): track 24.2 -> 22.9 mm
- added copper zone on F.Cu, net Net-(1206A_01x08_Male1-Pad1)
Other:
- net class Default: trace_width 0.5 -> 1
- board text removed: "4.5V"
